Commit message: add STL and such

File: catkin_ws/src/mmm_description/urdf/mmm.urdf.xacro (robot description, xacro)
@@ -1,127 +1,88 @@
 <?xml version="1.0"?>
-<robot name="arm" xmlns:xacro="http://www.ros.org/wiki/xacro">
-  <xacro:property name="PI" value="3.14159265359"/>
+<robot name="mmm" xmlns:xacro="http://www.ros.org/wiki/xacro">
+  <xacro:property name="PI" value="3.141592"/>
   <!-- Joints Control in Gazebo -->
   <gazebo>
     <plugin name="gazebo_ros_control" filename="libgazebo_ros_control.so"/>
   </gazebo>
-  <!-- Geometrical properties -->
-  <xacro:property name="link_side" value="0.02"/>
-  <xacro:property name="joint_radius" value="0.018"/>
-  <xacro:property name="joint_length" value="0.025"/>
-  <xacro:property name="toe_length" value="0.03"/>
-  <xacro:property name="foot_length" value="0.04"/>
-  <xacro:property name="leg_length" value="0.40"/>
-  <xacro:property name="arm_length" value="0.30"/>
-  <xacro:property name="hand_length" value="0.04"/>
-  <xacro:property name="finger_length" value="0.03"/>
+  <!-- macro to generate a link model -->
+  <!-- reads STL at mmm_description/meshes, and positions it at x,y,z -->
+  <xacro:macro name="create_link" params="index">
+    <link name="link${index}">
+      <visual>
+        <geometry>
+          <!-- the STL is exported from Fusion 360 in millimeters, while URDF expects it in meters.
+        Therefore, scaling is required. -->
+          <mesh scale="0.001 0.001 0.001" filename="package://mmm_description/meshes/link${index}.stl"/>
+        </geometry>
+        <material name="gray"/>
+      </visual>
+      <!--
+      <collision>
+      </collision>
+      <inertial>
+      </inertial> -->
+    </link>
+  </xacro:macro>
+  <!-- creates a link between link {index-1} and {index} -->
+  <!-- input distances in millimeters. -->
+  <xacro:macro name="create_joint" params="index x:=0 y:=0 z:=0 axis">
+    <joint name="link${index-1}_link${index}_joint" type="revolute">
+      <parent link="link${index-1}"/>
+      <child link="link${index}"/>
+      <origin xyz="${x/1000} ${y/1000} ${z/1000}"/>
+      <axis xyz="${axis}"/>
+      <limit
+        effort="40.0"
+        velocity="1.0"
+        lower="${-PI}"
+        upper="${PI}"/>
+    </joint>
+  </xacro:macro>
   <!-- Materials -->
-  <material name="orange">
-    <color rgba="1.00 0.67 0.02 1.00"/>
+  <material name="brown">
+    <color rgba="0.87 0.72 0.53 1.00"/>
   </material>
   <material name="gray">
-    <color rgba="0.80 0.80 0.80 1.00"/>
+    <color rgba="0.40 0.40 0.40 1.00"/>
   </material>
-  <!-- Generates a box visual/collision/inertial -->
-  <xacro:macro name="prism_vci" params="side length mass:=1 *origin">
-    <xacro:macro name="prism_geometry">
-      <xacro:insert_block name="origin"/>
+  <!-- World frame (for Gazebo) -->
+  <link name="world"/>
+  <!-- Base fixed to world frame -->
+  <joint name="world_base_joint" type="fixed">
+    <parent link="world"/>
+    <child link="base"/>
+  </joint>
+  <link name="base">
+    <visual>
+      <origin xyz="0 0 0" rpy="0 0 0"/>
       <geometry>
-        <box size="${side} ${side} ${length}"/>
+        <!-- the STL is exported from Fusion 360 in millimeters, while URDF expects it in meters.
+      Therefore, scaling is required. -->
+        <mesh scale="0.001 0.001 0.001" filename="package://mmm_description/meshes/base.stl"/>
       </geometry>
-    </xacro:macro>
-    <visual>
-      <xacro:prism_geometry/>
-      <material name="orange"/>
+      <material name="brown"/>
     </visual>
+    <!--
     <collision>
-      <xacro:prism_geometry/>
     </collision>
     <inertial>
-      <xacro:insert_block name="origin"/>
-      <mass value="${mass}"/>
-      <inertia ixx="${(mass/12)*(side*side+length*length)}"
-               iyy="${(mass/12)*(side*side+length*length)}"
-               izz="${(mass/6)*(side*side)}"
-               ixy="0" ixz="0" iyz="0"/>
-    </inertial>
-  </xacro:macro>
-  <!-- Generates a cylinder visual/collision -->
-  <xacro:macro name="cylinder_vc" params="radius length *origin">
-    <xacro:macro name="cylinder_geometry">
-      <xacro:insert_block name="origin"/>
-      <geometry>
-        <cylinder length="${length}" radius="${radius}"/>
-      </geometry>
-    </xacro:macro>
-    <visual>
-      <xacro:cylinder_geometry/>
-      <material name="gray"/>
-    </visual>
-    <collision>
-      <xacro:cylinder_geometry/>
-    </collision>
-  </xacro:macro>
-  <!-- Generates child joint of parent -->
-  <xacro:macro name="arm_joint" params="child parent dist:=0 axis">
-    <joint name="${parent}_${child}_joint" type="revolute">
-      <origin xyz="0 0 ${dist}" rpy="0 0 0"/>
-      <parent link="${parent}"/>
-      <child link="${child}"/>
-      <axis xyz="${axis}"/>
-      <limit effort="40.0"
-             velocity="1.0"
-             lower="${-PI}"
-             upper="${PI}"/>
-    </joint>
-    <!-- Required for ROS control -->
-    <transmission name="${parent}_${child}_transmission">
-      <type>transmission_interface/SimpleTransmission</type>
-      <joint name="${parent}_${child}_joint">
-        <hardwareInterface>hardware_interface/EffortJointInterface</hardwareInterface>
-      </joint>
-      <actuator name="${parent}_${child}_actuator"/>
-    </transmission>
-    <link name="${parent}">
-      <xacro:prism_vci length="${dist}" side="${link_side}">
-        <origin xyz="0 0 ${dist/2}" rpy="0 0 0"/>
-      </xacro:prism_vci>
-      <xacro:cylinder_vc radius="${joint_radius}" length="${joint_length}">
-        <xacro:if value="${axis=='0 0 1'}">
-          <origin xyz="0 0 ${dist}" rpy="0 0 0"/>
-        </xacro:if>
-        <xacro:if value="${axis=='1 0 0'}">
-          <origin xyz="0 0 ${dist}" rpy="0 ${PI/2} 0"/>
-        </xacro:if>
-        <xacro:if value="${axis=='0 1 0'}">
-          <origin xyz="0 0 ${dist}" rpy="${PI/2} 0 0"/>
-        </xacro:if>
-      </xacro:cylinder_vc>
-    </link>
-    <gazebo reference="${parent}">
-      <material>Gazebo/Orange</material>
-    </gazebo>
-  </xacro:macro>
-  <!-- World frame (for Gazebo) -->
-  <link name="world"/>
-  <!-- Arm fixed to world frame  -->
-  <joint name="world_foot_joint" type="fixed">
-    <parent link="world"/>
-    <child link="toe"/>
+    </inertial> -->
+  </link>
+  <joint name="base_link0_joint" type="fixed">
+    <parent link="base"/>
+    <child link="link0"/>
+    <origin xyz="${-30.2/1000} ${0/1000} ${6.9/1000}"/>
   </joint>
-  <!-- Joints Chain -->
-  <xacro:arm_joint parent="toe" child="foot" axis="0 0 1" dist="${toe_length}"/>
-  <xacro:arm_joint parent="foot" child="leg" axis="1 0 0" dist="${foot_length}"/>
-  <xacro:arm_joint parent="leg" child="arm" axis="1 0 0" dist="${leg_length}"/>
-  <xacro:arm_joint parent="arm" child="hand" axis="0 0 1" dist="${arm_length}"/>
-  <xacro:arm_joint parent="hand" child="finger" axis="1 0 0" dist="${hand_length}"/>
-  <!-- End effector -->
-  <link name="finger">
-    <xacro:prism_vci length="${finger_length}" side="${link_side}">
-      <origin xyz="0 0 ${finger_length/2}" rpy="0 0 0"/>
-    </xacro:prism_vci>
-  </link>
-  <gazebo reference="finger">
-    <material>Gazebo/Red</material>
-  </gazebo>
+  <xacro:create_link index="0"/>
+  <xacro:create_joint index="1" z="31" axis="0 0 1"/>
+  <xacro:create_link index="1"/>
+  <xacro:create_joint index="2" y="15.46" z="20.25" axis="0 1 0"/>
+  <xacro:create_link index="2"/>
+  <xacro:create_joint index="3" z="48" axis="0 1 0"/>
+  <xacro:create_link index="3"/>
+  <xacro:create_joint index="4" x="13.72" y="-15.5" z="53.22" axis="1 0 0"/>
+  <xacro:create_link index="4"/>
+  <xacro:create_joint index="5" x="-15.8" y="-15.9" z="40" axis="0 1 0"/>
+  <xacro:create_link index="5"/>
 </robot>

Commit message: change rviz.launch so it doesn't publish joints by itself add meshes and links in URDF

File: catkin_ws/src/mmm_description/urdf/mmm.urdf.xacro (robot description, xacro)
@@ -45,5 +45,5 @@
   </material>
   <material name="gray">
-    <color rgba="0.40 0.40 0.40 1.00"/>
+    <color rgba="0.90 0.90 0.90 1.00"/>
   </material>
   <!-- World frame (for Gazebo) -->
@@ -86,3 +86,35 @@
   <xacro:create_joint index="5" x="-15.8" y="-15.9" z="40" axis="0 1 0"/>
   <xacro:create_link index="5"/>
+  <xacro:create_joint index="6" y="13.9" z="69.5" axis="0 0 1"/>
+  <xacro:create_link index="6"/>
+  <xacro:create_joint index="7" y="-13.9" z="23.5" axis="0 1 0">
+  </xacro:create_joint>
+  <xacro:create_link index="7"/>
+  <joint name="link6_link7b_joint" type="revolute">
+    <parent link="link6"/>
+    <child link="link7b"/>
+    <origin xyz="${-20.97/1000} ${13.04/1000} ${34/1000}" rpy="0 0 ${PI}"/>
+    <axis xyz="0 1 0"/>
+    <limit
+      effort="40.0"
+      velocity="1.0"
+      lower="${-PI}"
+      upper="${PI}"/>
+    <mimic joint="link6_link7_joint" offset="${-PI*50/180}"/>
+  </joint>
+  <link name="link7b">
+    <visual>
+      <geometry>
+        <!-- the STL is exported from Fusion 360 in millimeters, while URDF expects it in meters.
+      Therefore, scaling is required. -->
+        <mesh scale="0.001 0.001 0.001" filename="package://mmm_description/meshes/link7.stl"/>
+      </geometry>
+      <material name="gray"/>
+    </visual>
+    <!--
+    <collision>
+    </collision>
+    <inertial>
+    </inertial> -->
+  </link>
 </robot>

Commit message: add raspicam_node package, add camera STL and edited URDF, add launch file

File: catkin_ws/src/mmm_description/urdf/mmm.urdf.xacro (robot description, xacro)
@@ -118,3 +118,24 @@
     </inertial> -->
   </link>
+  <joint name="link7b_camera_joint" type="fixed">
+    <parent link="link7b"/>
+    <child link="camera"/>
+    <origin xyz="${21/1000} ${14.93/1000} ${13.9/1000}" rpy="0 ${25*PI/180} 0"/>
+  </joint>
+  <link name="camera">
+    <visual>
+      <origin xyz="0 0 0" rpy="0 0 0"/>
+      <geometry>
+        <!-- the STL is exported from Fusion 360 in millimeters, while URDF expects it in meters.
+      Therefore, scaling is required. -->
+        <mesh scale="0.001 0.001 0.001" filename="package://mmm_description/meshes/camera.stl"/>
+      </geometry>
+      <material name="brown"/>
+    </visual>
+    <!--
+    <collision>
+    </collision>
+    <inertial>
+    </inertial> -->
+  </link>
 </robot>

Commit message: add moveit files

File: catkin_ws/src/mmm_description/urdf/mmm.urdf.xacro (robot description, xacro)
@@ -18,7 +18,12 @@
         <material name="gray"/>
       </visual>
-      <!--
       <collision>
+      <geometry>
+        <!-- the STL is exported from Fusion 360 in millimeters, while URDF expects it in meters.
+      Therefore, scaling is required. -->
+        <mesh scale="0.001 0.001 0.001" filename="package://mmm_description/meshes/Slink${index}.stl"/>
+      </geometry>
       </collision>
+<!--
       <inertial>
       </inertial> -->
@@ -27,5 +32,5 @@
   <!-- creates a link between link {index-1} and {index} -->
   <!-- input distances in millimeters. -->
-  <xacro:macro name="create_joint" params="index x:=0 y:=0 z:=0 axis">
+  <xacro:macro name="create_joint" params="index x:=0 y:=0 z:=0 axis angle">
     <joint name="link${index-1}_link${index}_joint" type="revolute">
       <parent link="link${index-1}"/>
@@ -36,6 +41,6 @@
         effort="40.0"
         velocity="1.0"
-        lower="${-PI}"
-        upper="${PI}"/>
+        lower="${-angle*PI/180}"
+        upper="${angle*PI/180}"/>
     </joint>
   </xacro:macro>
@@ -64,8 +69,12 @@
       <material name="brown"/>
     </visual>
-    <!--
     <collision>
+      <geometry>
+        <!-- the STL is exported from Fusion 360 in millimeters, while URDF expects it in meters.
+      Therefore, scaling is required. -->
+        <mesh scale="0.001 0.001 0.001" filename="package://mmm_description/meshes/Sbase.stl"/>
+      </geometry>
     </collision>
-    <inertial>
+    <!-- <inertial>
     </inertial> -->
   </link>
@@ -76,17 +85,24 @@
   </joint>
   <xacro:create_link index="0"/>
-  <xacro:create_joint index="1" z="31" axis="0 0 1"/>
+  <xacro:create_joint index="1" z="31" axis="0 0 1" angle="120"/>
   <xacro:create_link index="1"/>
-  <xacro:create_joint index="2" y="15.46" z="20.25" axis="0 1 0"/>
+  <xacro:create_joint index="2" y="15.46" z="20.25" axis="0 1 0" angle="60"/>
   <xacro:create_link index="2"/>
-  <xacro:create_joint index="3" z="48" axis="0 1 0"/>
+  <xacro:create_joint index="3" z="48" axis="0 1 0" angle="60"/>
   <xacro:create_link index="3"/>
-  <xacro:create_joint index="4" x="13.72" y="-15.5" z="53.22" axis="1 0 0"/>
+  <xacro:create_joint index="4" x="13.72" y="-15.5" z="53.22" axis="1 0 0" angle="90"/>
   <xacro:create_link index="4"/>
-  <xacro:create_joint index="5" x="-15.8" y="-15.9" z="40" axis="0 1 0"/>
+  <xacro:create_joint index="5" x="-15.8" y="-15.9" z="40" axis="0 1 0" angle="90"/>
   <xacro:create_link index="5"/>
-  <xacro:create_joint index="6" y="13.9" z="69.5" axis="0 0 1"/>
+  <xacro:create_joint index="6" y="13.9" z="69.5" axis="0 0 1" angle="135"/>
   <xacro:create_link index="6"/>
-  <xacro:create_joint index="7" y="-13.9" z="23.5" axis="0 1 0">
+  <joint name="link6_gripper_frame_joint" type="fixed">
+    <parent link="link6" />
+    <child link="gripper_frame"/>
+    <origin xyz="0 0 ${50/1000}"/>
+  </joint>
+  <link name="gripper_frame">
+  </link>
+  <xacro:create_joint index="7" y="-13.9" z="23.5" axis="0 1 0" angle="20">
   </xacro:create_joint>
   <xacro:create_link index="7"/>
@@ -112,8 +128,12 @@
       <material name="gray"/>
     </visual>
-    <!--
     <collision>
+      <geometry>
+        <!-- the STL is exported from Fusion 360 in millimeters, while URDF expects it in meters.
+      Therefore, scaling is required. -->
+        <mesh scale="0.001 0.001 0.001" filename="package://mmm_description/meshes/Slink7.stl"/>
+      </geometry>
     </collision>
-    <inertial>
+    <!-- <inertial>
     </inertial> -->
   </link>

Commit message: changes

File: catkin_ws/src/mmm_description/urdf/mmm.urdf.xacro (robot description, xacro)
@@ -140,8 +140,8 @@
   <joint name="link7b_camera_joint" type="fixed">
     <parent link="link7b"/>
-    <child link="camera"/>
+    <child link="raspicam"/>
     <origin xyz="${21/1000} ${14.93/1000} ${13.9/1000}" rpy="0 ${25*PI/180} 0"/>
   </joint>
-  <link name="camera">
+  <link name="raspicam">
     <visual>
       <origin xyz="0 0 0" rpy="0 0 0"/>

Commit message: fix camera origin

File: catkin_ws/src/mmm_description/urdf/mmm.urdf.xacro (robot description, xacro)
@@ -145,5 +145,5 @@
   <link name="raspicam">
     <visual>
-      <origin xyz="0 0 0" rpy="0 0 0"/>
+      <origin xyz="0 0 0" rpy="0 ${-PI/2} 0"/>
       <geometry>
         <!-- the STL is exported from Fusion 360 in millimeters, while URDF expects it in meters.

Commit message: fix camera again

File: catkin_ws/src/mmm_description/urdf/mmm.urdf.xacro (robot description, xacro)
@@ -141,5 +141,5 @@
     <parent link="link7b"/>
     <child link="raspicam"/>
-    <origin xyz="${21/1000} ${14.93/1000} ${13.9/1000}" rpy="0 ${25*PI/180} 0"/>
+    <origin xyz="${21/1000} ${14.93/1000} ${13.9/1000}" rpy="0 ${115*PI/180} 0"/>
   </joint>
   <link name="raspicam">

Commit message: various changes...

File: catkin_ws/src/mmm_description/urdf/mmm.urdf.xacro (robot description, xacro)
@@ -140,10 +140,10 @@
   <joint name="link7b_camera_joint" type="fixed">
     <parent link="link7b"/>
-    <child link="raspicam"/>
-    <origin xyz="${21/1000} ${14.93/1000} ${13.9/1000}" rpy="0 ${115*PI/180} 0"/>
+    <child link="camera"/>
+    <origin xyz="${21/1000} ${14.93/1000} ${13.9/1000}" rpy="0 ${25*PI/180} 0"/>
   </joint>
-  <link name="raspicam">
+  <link name="camera">
     <visual>
-      <origin xyz="0 0 0" rpy="0 ${-PI/2} 0"/>
+      <origin xyz="0 0 0" rpy="0 0 0"/>
       <geometry>
         <!-- the STL is exported from Fusion 360 in millimeters, while URDF expects it in meters.
@@ -159,3 +159,9 @@
     </inertial> -->
   </link>
+  <link name="raspicam"/>
+  <joint name="camera_raspicam_joint" type="fixed">
+    <parent link="camera"/>
+    <child link="raspicam"/>
+    <origin xyz="0 0 0" rpy="0 ${-PI/2} 0"/>
+  </joint>
 </robot>

Commit message: commit from Pi

File: catkin_ws/src/mmm_description/urdf/mmm.urdf.xacro (robot description, xacro)
@@ -163,5 +163,5 @@
     <parent link="camera"/>
     <child link="raspicam"/>
-    <origin xyz="0 0 0" rpy="0 ${-PI/2} 0"/>
+    <origin xyz="0 0 0" rpy="${PI/2} 0 ${PI/2}"/>
   </joint>
 </robot>

Commit message: fix: It all works on the new USB camera!

File: catkin_ws/src/mmm_description/urdf/mmm.urdf.xacro (robot description, xacro)
@@ -138,10 +138,10 @@
     </inertial> -->
   </link>
-  <joint name="link7b_camera_joint" type="fixed">
+  <joint name="link7b_camera_mesh_joint" type="fixed">
     <parent link="link7b"/>
-    <child link="camera"/>
+    <child link="camera_mesh"/>
     <origin xyz="${21/1000} ${14.93/1000} ${13.9/1000}" rpy="0 ${25*PI/180} 0"/>
   </joint>
-  <link name="camera">
+  <link name="camera_mesh">
     <visual>
       <origin xyz="0 0 0" rpy="0 0 0"/>
@@ -159,9 +159,9 @@
     </inertial> -->
   </link>
-  <link name="raspicam"/>
-  <joint name="camera_raspicam_joint" type="fixed">
-    <parent link="camera"/>
-    <child link="raspicam"/>
-    <origin xyz="0 0 0" rpy="${PI/2} 0 ${PI/2}"/>
+  <link name="camera"/>
+  <joint name="camera_mesh_camera_joint" type="fixed">
+    <parent link="camera_mesh"/>
+    <child link="camera"/>
+    <origin xyz="0 0 0" rpy="${-PI/2} 0 ${-PI/2}"/>
   </joint>
 </robot>
